Commit message: added huitao hw 3

File: HW3/Huitao/julia/odes/panda.urdf (robot description, URDF)
Before this commit: robot panda, 13 links, 12 joints
Links:
- link panda_hand: geometry collision mesh filename=meshes/collision/hand.obj; visual mesh filename=meshes/collision/hand.obj
- link panda_leftfinger: geometry collision mesh filename=meshes/collision/finger.obj; visual mesh filename=meshes/collision/finger.obj
- link panda_link0: geometry collision mesh filename=meshes/collision/link0.obj; visual mesh filename=meshes/collision/link0.obj
- link panda_link1: geometry collision mesh filename=meshes/collision/link1.obj; visual mesh filename=meshes/visual/link1.dae
- link panda_link2: geometry collision mesh filename=meshes/collision/link2.obj; visual mesh filename=meshes/visual/link2.dae
- link panda_link3: geometry collision mesh filename=meshes/collision/link3.obj; visual mesh filename=meshes/collision/link3.obj
- link panda_link4: geometry collision mesh filename=meshes/collision/link4.obj; visual mesh filename=meshes/collision/link4.obj
- link panda_link5: geometry collision mesh filename=meshes/collision/link5.obj; visual mesh filename=meshes/collision/link5.obj
- link panda_link6: geometry collision mesh filename=meshes/collision/link6.obj; visual mesh filename=meshes/visual/link6.dae
- link panda_link7: geometry collision mesh filename=meshes/collision/link7.obj; visual mesh filename=meshes/collision/link7.obj
- link panda_rightfinger: geometry collision mesh filename=meshes/collision/finger.obj; visual mesh filename=meshes/collision/finger.obj
